File: corne-chocolate/pcb/corne-chocolate.kicad_pcb (KiCad board)
At the start: 2 copper layers, 236.4 x 91.4 mm, 160 parts, among them J1 MJ-4PP-9, J2 Conn_01x04, J3 MJ-4PP-9, J4 Conn_01x04, P1 Conn_01x01, P2 Conn_01x01, P3 Conn_01x01, P4 Conn_01x01, SW10 SW_PUSH, SW11 SW_PUSH, SW12 SW_PUSH, SW13 SW_PUSH, SW14 SW_PUSH, SW15 SW_PUSH, SW16 SW_PUSH, SW17 SW_PUSH, SW18 SW_PUSH, SW19 SW_PUSH, SW2 SW_PUSH, SW20 SW_PUSH, SW21 SW_PUSH, SW22 SW_PUSH, SW23 SW_PUSH, SW24 SW_PUSH, SW25 SW_PUSH, SW26 SW_PUSH, SW27 SW_PUSH, SW28 SW_PUSH, SW29 SW_PUSH, SW3 SW_PUSH, SW30 SW_PUSH, SW31 SW_PUSH, SW32 SW_PUSH, SW33 SW_PUSH, SW34 SW_PUSH, SW35 SW_PUSH, SW36 SW_PUSH, SW37 SW_PUSH, SW4 SW_PUSH, SW5 SW_PUSH, SW6 SW_PUSH, SW7 SW_PUSH, SW8 SW_PUSH, SW9 SW_PUSH, U1 ProMicro, U2 ProMicro

Commit message: several important fixes
Parts:
- removed the J1 at (145.3, 112.8)
- removed JP2, JP3, JP4, JP5, JP6, JP7, JP8, JP9: Device:Jumper_NO_Small, kbd:Jumper
- removed L10, L11, L12, L13, L14, L15, L16, L17, L18, L19, L2, L20, L21, L3, L30, L31, L32, L33, L36, L37, L38, L39, L4, L40, L41, L42, L43, L46, L47, L48, L49, L5, L6, L7, L8, L9: SK6812MINI, kbd:YS-SK6812MINI-E
- removed L22, L23, L24, L25, L26, L27, L28, L29, L34, L35, L44, L45: SK6812MINI, kbd:SK6812MINI_underglow_rev
- removed the P2 at (131.6, 106.4)
- removed P3: Conn_01x01, kbd:1pin_conn
- added J2: 54-00174, kbd:54-00174_TEN, F.Cu at (145.4, 112.8)
- added LED1: YS-SK6812MINI-E, kbd:LED_SK6812-MINI-E, B.Cu at (39.6, 67.7)
- added LED10: YS-SK6812MINI-E, kbd:LED_SK6812-MINI-E, B.Cu at (77.6, 79.6)
- added LED11: YS-SK6812MINI-E, kbd:LED_SK6812-MINI-E, B.Cu at (96.6, 81.7)
- added LED12: WS2812B, kbd:LED_WS2812B_PLCC4_5.0x5.0mm_P3.2mm, B.Cu at (108.6, 84.6)
- added LED13: YS-SK6812MINI-E, kbd:LED_SK6812-MINI-E, B.Cu at (115.6, 84.1)
- added LED14: YS-SK6812MINI-E, kbd:LED_SK6812-MINI-E, B.Cu at (39.6, 105.7)
- added LED15: WS2812B, kbd:LED_WS2812B_PLCC4_5.0x5.0mm_P3.2mm, B.Cu at (51.2, 96.5)
- added LED16: YS-SK6812MINI-E, kbd:LED_SK6812-MINI-E, B.Cu at (58.6, 101.0)
- added LED17: YS-SK6812MINI-E, kbd:LED_SK6812-MINI-E, B.Cu at (77.6, 98.6)
- added LED18: YS-SK6812MINI-E, kbd:LED_SK6812-MINI-E, B.Cu at (96.6, 101.0)
- added LED19: YS-SK6812MINI-E, kbd:LED_SK6812-MINI-E, B.Cu at (115.6, 103.4)
- added LED2: YS-SK6812MINI-E, kbd:LED_SK6812-MINI-E, B.Cu at (58.7, 63.0)
- added LED20: WS2812B, kbd:LED_WS2812B_PLCC4_5.0x5.0mm_P3.2mm, B.Cu at (79.2, 118.3)
- added LED21: YS-SK6812MINI-E, kbd:LED_SK6812-MINI-E, B.Cu at (87.1, 120.6)
- added LED22: YS-SK6812MINI-E, kbd:LED_SK6812-MINI-E, B.Cu at (109.7, 123.6)
- added LED23: WS2812B, kbd:LED_WS2812B_PLCC4_5.0x5.0mm_P3.2mm, B.Cu at (119.2, 121.3)
- added LED24: YS-SK6812MINI-E, kbd:LED_SK6812-MINI-E, B.Cu at (125.7, 129.9)
- added LED25: YS-SK6812MINI-E, kbd:LED_SK6812-MINI-E, B.Cu at (179.7, 65.4)
- added LED26: YS-SK6812MINI-E, kbd:LED_SK6812-MINI-E, B.Cu at (198.7, 63.0)
- added LED27: YS-SK6812MINI-E, kbd:LED_SK6812-MINI-E, B.Cu at (217.7, 60.6)
- added LED28: YS-SK6812MINI-E, kbd:LED_SK6812-MINI-E, B.Cu at (236.7, 63.0)
- added LED29: YS-SK6812MINI-E, kbd:LED_SK6812-MINI-E, B.Cu at (255.7, 67.7)
- added LED3: YS-SK6812MINI-E, kbd:LED_SK6812-MINI-E, B.Cu at (77.6, 60.6)
- added LED30: WS2812B, kbd:LED_WS2812B_PLCC4_5.0x5.0mm_P3.2mm, B.Cu at (172.4, 84.4)
- added LED31: YS-SK6812MINI-E, kbd:LED_SK6812-MINI-E, B.Cu at (179.7, 84.3)
- added LED32: YS-SK6812MINI-E, kbd:LED_SK6812-MINI-E, B.Cu at (198.7, 82.0)
- added LED33: WS2812B, kbd:LED_WS2812B_PLCC4_5.0x5.0mm_P3.2mm, B.Cu at (209.9, 80.6)
- added LED34: YS-SK6812MINI-E, kbd:LED_SK6812-MINI-E, B.Cu at (217.7, 79.6)
- added LED35: YS-SK6812MINI-E, kbd:LED_SK6812-MINI-E, B.Cu at (236.7, 82.0)
- added LED36: WS2812B, kbd:LED_WS2812B_PLCC4_5.0x5.0mm_P3.2mm, B.Cu at (247.9, 88.1)
- added LED37: YS-SK6812MINI-E, kbd:LED_SK6812-MINI-E, B.Cu at (255.7, 86.7)
- added LED38: YS-SK6812MINI-E, kbd:LED_SK6812-MINI-E, B.Cu at (179.7, 103.4)
- added LED39: YS-SK6812MINI-E, kbd:LED_SK6812-MINI-E, B.Cu at (198.7, 101.0)
- added LED4: YS-SK6812MINI-E, kbd:LED_SK6812-MINI-E, B.Cu at (96.7, 63.0)
- added LED40: YS-SK6812MINI-E, kbd:LED_SK6812-MINI-E, B.Cu at (217.7, 98.6)
- added LED41: YS-SK6812MINI-E, kbd:LED_SK6812-MINI-E, B.Cu at (236.7, 101.0)
- added LED42: WS2812B, kbd:LED_WS2812B_PLCC4_5.0x5.0mm_P3.2mm, B.Cu at (247.9, 107.1)
- added LED43: YS-SK6812MINI-E, kbd:LED_SK6812-MINI-E, B.Cu at (255.7, 105.7)
- added LED44: YS-SK6812MINI-E, kbd:LED_SK6812-MINI-E, B.Cu at (169.7, 129.9)
- added LED45: WS2812B, kbd:LED_WS2812B_PLCC4_5.0x5.0mm_P3.2mm, B.Cu at (173.2, 121.6)
- added LED46: YS-SK6812MINI-E, kbd:LED_SK6812-MINI-E, B.Cu at (185.7, 123.6)
- added LED47: YS-SK6812MINI-E, kbd:LED_SK6812-MINI-E, B.Cu at (208.3, 120.6)
- added LED48: WS2812B, kbd:LED_WS2812B_PLCC4_5.0x5.0mm_P3.2mm, B.Cu at (215.1, 116.3)
- added LED5: YS-SK6812MINI-E, kbd:LED_SK6812-MINI-E, B.Cu at (115.6, 65.4)
- added LED6: WS2812B, kbd:LED_WS2812B_PLCC4_5.0x5.0mm_P3.2mm, B.Cu at (50.7, 77.6)
- added LED7: YS-SK6812MINI-E, kbd:LED_SK6812-MINI-E, B.Cu at (39.6, 86.7)
- added LED8: YS-SK6812MINI-E, kbd:LED_SK6812-MINI-E, B.Cu at (58.6, 82.0)
- added LED9: WS2812B, kbd:LED_WS2812B_PLCC4_5.0x5.0mm_P3.2mm, B.Cu at (70.4, 79.9)
- D1: renamed from D2; moved to B.Cu
- D10: renamed from D12; moved to B.Cu
- D11: renamed from D14; moved to B.Cu
- D12: renamed from D15; moved to B.Cu
- D13: renamed from D16; moved to B.Cu
- D14: renamed from D17; moved to B.Cu
- D15: renamed from D18; moved to B.Cu
- D16: renamed from D19; moved to B.Cu
- D17: renamed from D20; moved to B.Cu
- D18: renamed from D21; moved to B.Cu
- D19: renamed from D7; moved to B.Cu
- D2: renamed from D3; moved to B.Cu
- D20: renamed from D23; moved to B.Cu
- D21: renamed from D26; moved to B.Cu
- D22: renamed from D30; moved to B.Cu
- D23: renamed from D34; moved to B.Cu
- D24: renamed from D13; moved to B.Cu
- D25: renamed from D24; moved to B.Cu
- D26: renamed from D27; moved to B.Cu
- D27: renamed from D31; moved to B.Cu
- D28: renamed from D35; moved to B.Cu
- D29: renamed from D22; moved to B.Cu
- D3: renamed from D4; moved to B.Cu
- D30: renamed from D25; moved to B.Cu
- D31: renamed from D28; moved to B.Cu
- D32: moved to B.Cu
- D33: renamed from D36; moved to B.Cu
- D34: renamed from D29; moved to B.Cu
- D35: renamed from D33; moved to B.Cu
- D36: renamed from D37; moved to B.Cu
- D4: renamed from D5; moved to B.Cu
- D5: renamed from D6; moved to B.Cu
- D6: renamed from D8; moved to B.Cu
- D7: renamed from D9; moved to B.Cu
- D8: renamed from D10; moved to B.Cu
- D9: renamed from D11; moved to B.Cu
- J3: value MJ-4PP-9 -> 781271220; footprint kbd:MJ-4PP-9_1side -> kbd:CON_781271220
- J4: value Conn_01x04 -> 54-00174; footprint kbd:OLED_1side -> kbd:54-00174_TEN
- R1, R2: footprint kbd:R -> Resistor_SMD:R_1206_3216Metric_Pad1.30x1.75mm_HandSolder
- R3, R4: value R -> 4k7; footprint kbd:R -> kbd:R_1206_3216Metric_Pad1.30x1.75mm_HandSolder
- moved D18 39.4 mm to (137.2, 129.4), turned to -30 degrees
- moved D36 37.0 mm to (164.2, 140.3), turned to -150 degrees
- moved D17 22.3 mm to (113.8, 136.2), turned to 165 degrees
- moved D5 18.4 mm to (121.6, 78.4), turned to 90 degrees
- moved D10 18.3 mm to (121.7, 97.3), turned to 90 degrees
- moved D15 18.1 mm to (121.6, 116.0), turned to 90 degrees
- moved J4 17.6 mm to (150.0, 112.8), turned to 90 degrees
- moved D25 17.0 mm to (242.8, 95.1), turned to 90 degrees
- moved D24 17.0 mm to (261.8, 99.8), turned to 90 degrees
- moved D16 16.9 mm to (94.1, 132.0), turned to 180 degrees
- moved D30 16.9 mm to (242.8, 113.8), turned to 90 degrees
- moved D21 16.9 mm to (223.7, 73.6), turned to 90 degrees
- moved D22 16.9 mm to (204.7, 75.9), turned to 90 degrees
- moved D19 16.8 mm to (261.8, 80.6), turned to 90 degrees
- moved D20 16.8 mm to (242.8, 75.8), turned to 90 degrees
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- renumbered H11 to H10, H13 to H11, H14 to H12, H9 to H13, H8 to H14, H5 to H3, H6 to H4, H7 to H5, H4 to H6, H3 to H7, H10 to H8, H12 to H9, J2 to J1, P4 to P2, SW2 to SW1, SW12 to SW10, SW14 to SW11, SW15 to SW12, SW16 to SW13, SW17 to SW14, SW18 to SW15, SW19 to SW16, SW20 to SW17, SW21 to SW18, SW7 to SW19, SW3 to SW2, SW23 to SW20, SW26 to SW21, SW30 to SW22, SW34 to SW23, SW13 to SW24, SW24 to SW25, SW27 to SW26, SW31 to SW27, SW35 to SW28, SW22 to SW29, SW4 to SW3, SW25 to SW30, SW28 to SW31, SW36 to SW33, SW29 to SW34, SW33 to SW35, SW37 to SW36, SW5 to SW4, SW6 to SW5, SW8 to SW6, SW9 to SW7, SW10 to SW8, SW11 to SW9
Connections:
- J1 pad 1: Net-(J2-Pin_1) -> LSDA
- J1 pad 2: Net-(J2-Pin_2) -> LSCL
- J1 pad 3: Net-(J2-Pin_3) -> LVCC
- J1 pad 4: Net-(J2-Pin_4) -> LGND
- J4 pad 1: Net-(J4-Pin_1) -> RGND
- J4 pad 2: Net-(J4-Pin_2) -> RVCC
- J4 pad 3: Net-(J4-Pin_3) -> unconnected-(J4-Pad3)
- J4 pad 4: Net-(J4-Pin_4) -> Rdata
- P1 pad 1: Net-(P1-Pin_1) -> Ldata
Routing:
- net LGND: track 627.4 -> 528.4 mm, vias 42 -> 10
- net Net-(LED43-DOUT): track 0.00 -> 66.0 mm
- net Net-(LED14-DOUT): track 0.00 -> 57.4 mm
- net Net-(D18-A): track 57.8 -> 3.08 mm
- net Net-(L25-DOUT): track 53.6 -> 0.00 mm
- net Net-(L29-DOUT): track 52.6 -> 0.00 mm, vias 2 -> 0
- net RVCC: track 540.7 -> 490.9 mm, vias 9 -> 6
- net RGND: track 497.3 -> 543.5 mm, vias 30 -> 4
- net Net-(L28-DIN): track 41.4 -> 0.00 mm
- net Net-(L17-DOUT): track 40.5 -> 0.00 mm, vias 2 -> 0
- net Net-(L23-DIN): track 40.1 -> 0.00 mm, vias 2 -> 0
- net Net-(L26-DOUT): track 39.9 -> 0.00 mm
- net Net-(D36-A): track 42.1 -> 3.22 mm
- net Net-(L48-DIN): track 38.1 -> 0.00 mm, vias 2 -> 0
- net Net-(L22-DIN): track 36.3 -> 0.00 mm
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- added copper zone on F.Cu, net Lcol2
- added copper zone on F.Cu, net Lcol3
- added copper zone on F.Cu, net Lcol5
- added copper zone on F.Cu, net Rcol1
- added copper zone on F.Cu, net Rcol2
- added copper zone on F.Cu, net Rcol3
- added copper zone on F.Cu, net Rcol4
- added copper zone on F.Cu, net Rcol5
- removed copper zone on B.Cu, net (none)
- removed copper zone on B.Cu, net LGND
- removed copper zone on F.Cu, net LGND
- removed copper zone on B.Cu, net LVCC
- removed copper zone on F.Cu, net LVCC
- removed copper zone on B.Cu, net Lrow2
Other:
- board text removed: "Designed by foostan Remixed by ektocommers"
